File: rmk-ble-keyboard.kicad_pcb (KiCad board)
At the start: 2 copper layers, 301.2 x 94.1 mm, 165 parts, among them J2 JST_SH_SM04B-SRSS-TB, J4 Debug, J5 RGB, Q1 Si2301CDS, SW1 esc, SW10 9, SW11 0, SW12 -, SW13 =, SW14 backspace, SW15 del, SW16 tab, SW17 q, SW18 w, SW19 e, SW2 1, SW20 r, SW21 t, SW22 y, SW23 u, SW24 i, SW25 o, SW26 p, SW27 [, SW28 ], SW29 \, SW3 2, SW30 pgup, SW31 capslock, SW32 a, SW33 s, SW34 d, SW35 f, SW36 g, SW37 h, SW38 j, SW39 k, SW4 3, SW40 l, SW41 ;, SW42 ', SW43 enter, SW44 pgdn, SW45 lshift, SW46 z, SW47 x, SW48 c, SW49 v, SW5 4, SW50 b, SW51 n, SW52 m, SW53 ,, SW54 ., SW55 /, SW56 rshift, SW57 up, SW58 fn, SW59 lctrl, SW6 5, SW60 lgui, SW61 lalt, SW62 space, SW63 ralt, SW64 menu, SW65 left, SW66 down, SW67 right, SW68 SW_Push, SW7 6, SW8 7, SW9 8, U1 TP4056, Y1 32.768KHZ

Commit message: feat: update pcb and firmware and readme
Signed-off-by: HaoboGu <haobogu@outlook.com>
Connections:
- U4 pad 18: unconnected-(U4-AI2-Pad18) -> /mcu/caps
Routing:
- net /mcu/caps: track 0.00 -> 177.6 mm, vias 0 -> 5
- net /mcu/Li+: track 159.2 -> 160.5 mm
- net GND: vias 86 -> 96
